File: attiny85.brd (EAGLE design)
At the start: 74.7 x 55.5 mm, 8 parts, among them U1 TINY85-20-DIP

Commit message: More fixing of values
Parts:
- R17, R18: value 1M -> 1MΩ
Changed lines of the file:
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@@
 <attribute name="VALUE" x="19.7104" y="7.8486" size="1.27" layer="27" ratio="10"/>
 </element>
-<element name="R17" library="SparkFun-Resistors" package="AXIAL-0.3" value="1M" x="29.845" y="33.02" rot="R270">
+<element name="R17" library="SparkFun-Resistors" package="AXIAL-0.3" value="1MΩ" x="29.845" y="33.02" rot="R270">
 <attribute name="VALUE" value="1k" x="29.845" y="33.02" size="1.778" layer="27" rot="R270" display="off"/>
 <attribute name="PROD_ID" value="RES-08380" x="29.845" y="33.02" size="1.778" layer="27" rot="R270" display="off"/>
 </element>
-<element name="R18" library="SparkFun-Resistors" package="AXIAL-0.3" value="1M" x="27.94" y="19.05" rot="R45">
+<element name="R18" library="SparkFun-Resistors" package="AXIAL-0.3" value="1MΩ" x="27.94" y="19.05" rot="R45">
 <attribute name="VALUE" value="1k" x="27.94" y="19.05" size="1.778" layer="27" rot="R45" display="off"/>
 <attribute name="PROD_ID" value="RES-08380" x="27.94" y="19.05" size="1.778" layer="27" rot="R45" display="off"/>

Commit message: Adjusting a routing issue
Routing:
- net CAP1: track 52.8 -> 50.8 mm
Changed lines of the file:
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@@
 <setting verticaltext="up"/>
 </settings>
-<grid distance="0.05" unitdist="inch" unit="mm" style="lines" multiple="1" display="yes" altdistance="0.00125" altunitdist="inch" altunit="mm"/>
+<grid distance="0.05" unitdist="inch" unit="inch" style="lines" multiple="1" display="yes" altdistance="0.0125" altunitdist="mm" altunit="mm"/>
 <layers>
 <layer number="1" name="Top" color="4" fill="1" visible="yes" active="yes"/>
@@
 <wire x1="36.60775" y1="21.24075" x2="34.70275" y2="19.20875" width="0.4064" layer="1"/>
 <wire x1="34.70275" y1="19.20875" x2="31.6865" y2="16.383" width="0.4064" layer="1"/>
-<wire x1="31.6865" y1="16.383" x2="29.05125" y2="14.31925" width="0.4064" layer="1"/>
-<wire x1="29.05125" y1="14.31925" x2="27.40025" y2="13.17625" width="0.4064" layer="1"/>
+<wire x1="31.6865" y1="16.383" x2="30.3838125" y2="15.362821875" width="0.4064" layer="1"/>
 <via x="33.3375" y="26.035" extent="1-16" drill="0.3048"/>
 <wire x1="33.3375" y1="26.035" x2="33.3375" y2="26.3525" width="0.4064" layer="1"/>
@@
 <wire x1="35.2425" y1="28.2575" x2="35.2425" y2="26.9875" width="0.4064" layer="1"/>
 <wire x1="35.2425" y1="26.9875" x2="36.83" y2="25.4" width="0.4064" layer="1"/>
-<wire x1="27.40025" y1="13.17625" x2="25.245921875" y2="16.355921875" width="0.4064" layer="1"/>
 <wire x1="13.97" y1="38.1" x2="19.05" y2="33.02" width="0.4064" layer="16"/>
 <wire x1="19.05" y1="33.02" x2="29.21" y2="33.02" width="0.4064" layer="16"/>
 <wire x1="29.21" y1="33.02" x2="33.3375" y2="28.8925" width="0.4064" layer="16"/>
 <wire x1="33.3375" y1="28.8925" x2="33.3375" y2="26.035" width="0.4064" layer="16"/>
+<wire x1="25.245921875" y1="16.355921875" x2="26.67" y2="15.24" width="0.4064" layer="1"/>
+<wire x1="26.67" y1="15.24" x2="30.3838125" y2="15.362821875" width="0.4064" layer="1" curve="79.953522"/>
 </signal>
 <signal name="SENSE">
